Commit message: update: update nesfr_arm.urdf.xacro
Signed-off-by: Jaeyoung Lee <jylee0121@gmail.com>

File: nesfr_arm_description/urdf/nesfr_arm.urdf.xacro (robot description, xacro)
@@ -24,15 +24,61 @@
         <color rgba="0.1 0.1 0.1 1" />
     </material>
-    <link name="base_footprint"/>
-    <joint name="base_joint" type="fixed">
-        <parent link="base_footprint"/>
-        <child link="base_link"/>
-        <origin xyz="0.0 0.0 0.07131916" rpy="0 0 0"/>
+    <link name="robot_arm_base_footprint"/>
+    <link name="upper_arm_link">
+        <visual>
+            <origin xyz="0.0 0.0 0.15" rpy="0 0 0"/>
+            <geometry>
+                <box size="0.05 0.05 0.3" />
+            </geometry>
+            <material name="white"/>
+        </visual>
+        <collision>
+            <origin xyz="0.0 0.0 0.15" rpy="0 0 0"/>
+            <geometry>
+                <box size="0.05 0.05 0.3" />
+            </geometry>
+        </collision>
+    </link>
+    <link name="fore_arm_link">
+        <visual>
+            <origin xyz="0.0 0.0 0.15" rpy="0 0 0"/>
+            <geometry>
+                <box size="0.05 0.05 0.3" />
+            </geometry>
+            <material name="white"/>
+        </visual>
+        <collision>
+            <origin xyz="0.0 0.0 0.15" rpy="0 0 0"/>
+            <geometry>
+                <box size="0.05 0.05 0.3" />
+            </geometry>
+        </collision>
+    </link>
+    <joint name="shoulder_lift" type="revolute">
+        <parent link="robot_arm_base_footprint"/>
+        <child link="upper_arm_link"/>
+        <axis xyz="0 1 0" />
+        <limit effort="10" velocity="1"  lower="${-55.0*M_PI/180.0}" upper="0.0" />
+        <origin xyz="0.0 0.0 0.1" rpy="0 ${-5.0*M_PI/180.0} 0"/>
     </joint>
-    <link name="base_link">
+    <joint name="elbow_joint" type="revolute">
+        <parent link="upper_arm_link"/>
+        <child link="fore_arm_link"/>
+        <axis xyz="0 1 0" />
+        <limit effort="10" velocity="1"  lower="0.0" upper="${110.0*M_PI/180.0}" />
+        <origin xyz="0.0 0.0 0.3" rpy="0 ${10.0*M_PI/180.0} 0"/>
+    </joint>
+    <joint name="gimbal_base_joint" type="revolute">
+        <parent link="fore_arm_link"/>
+        <child link="gimbal_base_link"/>
+        <axis xyz="0 1 0" />
+        <limit effort="10" velocity="1"  lower="${-55.0*M_PI/180.0}" upper="0.0" />
+        <origin xyz="0.0 0.0 0.3" rpy="0 ${-5.0*M_PI/180.0} 0"/>
+    </joint>
+    <link name="gimbal_base_link">
         <visual>
             <origin xyz="0.0 0.0 0.05" rpy="0 0 0"/>
             <geometry>
-                <cylinder length="0.10" radius="0.10"/>
+                <cylinder length="0.10" radius="0.03"/>
             </geometry>
             <material name="white"/>
@@ -41,10 +87,10 @@
             <origin xyz="0.0 0.0 0.0" rpy="0 0 0"/>
             <geometry>
-                <cylinder length="0.10" radius="0.10"/>
+                <cylinder length="0.10" radius="0.03"/>
             </geometry>
         </collision>
     </link>
     <joint name="main_cam_base_joint" type="prismatic">
-        <parent link="base_link"/>
+        <parent link="gimbal_base_link"/>
         <child link="main_cam_pan_link"/>
         <axis xyz="0 0 1" />
@@ -70,5 +116,5 @@
         <child link="main_cam_link"/>
         <axis xyz="0 1 0" />
-        <limit effort="10" velocity="1"  lower="-${0.5*M_PI}" upper="0.0" />
+        <limit effort="10" velocity="1"  lower="-${0.5*M_PI}" upper="${0.5*M_PI}" />
         <origin xyz="0.0 0.0 0.0" rpy="0 0 0"/>
     </joint>

Commit message: update: update nesfr robot arm urdf and its constraints
Signed-off-by: Jaeyoung Lee <jylee0121@gmail.com>

File: nesfr_arm_description/urdf/nesfr_arm.urdf.xacro (robot description, xacro)
@@ -1,5 +1,41 @@
 <?xml version="1.0"?>
-<robot xmlns:xacro="http://wiki.ros.org/xacro" name="nesfr_arm_only" >
+<robot xmlns:xacro="http://wiki.ros.org/xacro" name="nesfr_arm" >
     <xacro:property name="M_PI" value="3.1415926535897931" />
+    <!--
+      reference: https://answers.ros.org/question/401950/ros2-any-idea-on-how-to-pass-parameters-yaml-to-a-xacro-file-via-launch-python-script/
+    -->
+    <xacro:arg name="nesfr_arm_params" default=""/>
+    <xacro:property name="nesfr_arm_params_file" value="$(arg nesfr_arm_params)"/>
+    <xacro:property name="nesfr_arm_parameters" value="${load_yaml(nesfr_arm_params_file)}"/>
+    <xacro:property name="shoulder_lift_lower_limit" value="${nesfr_arm_parameters['joint_limits']['shoulder_lift']['min_position']}"/>
+    <xacro:property name="shoulder_lift_upper_limit" value="${nesfr_arm_parameters['joint_limits']['shoulder_lift']['max_position']}"/>
+    <xacro:property name="elbow_joint_lower_limit" value="${nesfr_arm_parameters['joint_limits']['elbow_joint']['min_position']}"/>
+    <xacro:property name="elbow_joint_upper_limit" value="${nesfr_arm_parameters['joint_limits']['elbow_joint']['max_position']}"/>
+    <xacro:property name="wrist_joint_lower_limit" value="${nesfr_arm_parameters['joint_limits']['wrist_joint']['min_position']}"/>
+    <xacro:property name="wrist_joint_upper_limit" value="${nesfr_arm_parameters['joint_limits']['wrist_joint']['max_position']}"/>
+    <xacro:property name="upper_arm_x" value="${nesfr_arm_parameters['kinematics']['upper_arm']['x']}" />
+    <xacro:property name="upper_arm_y" value="${nesfr_arm_parameters['kinematics']['upper_arm']['y']}" />
+    <xacro:property name="upper_arm_z" value="${nesfr_arm_parameters['kinematics']['upper_arm']['z']}" />
+    <xacro:property name="upper_arm_roll" value="${nesfr_arm_parameters['kinematics']['upper_arm']['roll']}" />
+    <xacro:property name="upper_arm_pitch" value="${nesfr_arm_parameters['kinematics']['upper_arm']['pitch']}" />
+    <xacro:property name="upper_arm_yaw" value="${nesfr_arm_parameters['kinematics']['upper_arm']['yaw']}" />
+    <xacro:property name="fore_arm_x" value="${nesfr_arm_parameters['kinematics']['fore_arm']['x']}" />
+    <xacro:property name="fore_arm_y" value="${nesfr_arm_parameters['kinematics']['fore_arm']['y']}" />
+    <xacro:property name="fore_arm_z" value="${nesfr_arm_parameters['kinematics']['fore_arm']['z']}" />
+    <xacro:property name="fore_arm_roll" value="${nesfr_arm_parameters['kinematics']['fore_arm']['roll']}" />
+    <xacro:property name="fore_arm_pitch" value="${nesfr_arm_parameters['kinematics']['fore_arm']['pitch']}" />
+    <xacro:property name="fore_arm_yaw" value="${nesfr_arm_parameters['kinematics']['fore_arm']['yaw']}" />
+    <xacro:property name="upper_arm_x" value="${nesfr_arm_parameters['kinematics']['upper_arm']['x']}" />
+    <xacro:property name="upper_arm_y" value="${nesfr_arm_parameters['kinematics']['upper_arm']['y']}" />
+    <xacro:property name="upper_arm_z" value="${nesfr_arm_parameters['kinematics']['upper_arm']['z']}" />
+    <xacro:property name="upper_arm_roll" value="${nesfr_arm_parameters['kinematics']['upper_arm']['roll']}" />
+    <xacro:property name="upper_arm_pitch" value="${nesfr_arm_parameters['kinematics']['upper_arm']['pitch']}" />
+    <xacro:property name="upper_arm_yaw" value="${nesfr_arm_parameters['kinematics']['upper_arm']['yaw']}" />
+    <xacro:property name="wrist_x" value="${nesfr_arm_parameters['kinematics']['wrist']['x']}" />
+    <xacro:property name="wrist_y" value="${nesfr_arm_parameters['kinematics']['wrist']['y']}" />
+    <xacro:property name="wrist_z" value="${nesfr_arm_parameters['kinematics']['wrist']['z']}" />
+    <xacro:property name="wrist_roll" value="${nesfr_arm_parameters['kinematics']['wrist']['roll']}" />
+    <xacro:property name="wrist_pitch" value="${nesfr_arm_parameters['kinematics']['wrist']['pitch']}" />
+    <xacro:property name="wrist_yaw" value="${nesfr_arm_parameters['kinematics']['wrist']['yaw']}" />
     <xacro:property name="rgbd_cam_size_x" value="0.1" />
     <xacro:property name="rgbd_cam_size_y" value="0.2" />
@@ -24,5 +60,6 @@
         <color rgba="0.1 0.1 0.1 1" />
     </material>
-    <link name="robot_arm_base_footprint"/>
+    <link name="base_link"/>
+    <link name="robot_arm_base_link"/>
     <link name="upper_arm_link">
         <visual>
@@ -55,10 +92,44 @@
         </collision>
     </link>
+    <link name="wrist_link">
+        <visual>
+            <origin xyz="0.0 0.0 0.025" rpy="0 0 0"/>
+            <geometry>
+                <box size="0.05 0.05 0.05" />
+            </geometry>
+            <material name="white"/>
+        </visual>
+        <collision>
+            <origin xyz="0.0 0.0 0.025" rpy="0 0 0"/>
+            <geometry>
+                <box size="0.05 0.05 0.05" />
+            </geometry>
+        </collision>
+      </link>
+    <link name="gimbal_base_link">
+        <visual>
+            <origin xyz="0.0 0.0 0.05" rpy="0 0 0"/>
+            <geometry>
+                <cylinder length="0.10" radius="0.03"/>
+            </geometry>
+            <material name="white"/>
+        </visual>
+        <collision>
+            <origin xyz="0.0 0.0 0.0" rpy="0 0 0"/>
+            <geometry>
+                <cylinder length="0.10" radius="0.03"/>
+            </geometry>
+        </collision>
+    </link>
+    <joint name="base-robot_arm_base_fixed_joint" type="fixed">
+        <parent link="base_link"/>
+        <child link="robot_arm_base_link"/>
+    </joint>
     <joint name="shoulder_lift" type="revolute">
-        <parent link="robot_arm_base_footprint"/>
+        <parent link="robot_arm_base_link"/>
         <child link="upper_arm_link"/>
         <axis xyz="0 1 0" />
-        <limit effort="10" velocity="1"  lower="${-55.0*M_PI/180.0}" upper="0.0" />
-        <origin xyz="0.0 0.0 0.1" rpy="0 ${-5.0*M_PI/180.0} 0"/>
+        <limit effort="10" velocity="1"  lower="${shoulder_lift_lower_limit}" upper="${shoulder_lift_upper_limit}" />
+        <origin xyz="${upper_arm_x} ${upper_arm_y} ${upper_arm_z}" rpy="${upper_arm_roll} ${upper_arm_pitch} ${upper_arm_yaw}"/>
     </joint>
     <joint name="elbow_joint" type="revolute">
@@ -66,29 +137,19 @@
         <child link="fore_arm_link"/>
         <axis xyz="0 1 0" />
-        <limit effort="10" velocity="1"  lower="0.0" upper="${110.0*M_PI/180.0}" />
-        <origin xyz="0.0 0.0 0.3" rpy="0 ${10.0*M_PI/180.0} 0"/>
-    </joint>
-    <joint name="gimbal_base_joint" type="revolute">
+        <limit effort="10" velocity="1"  lower="${elbow_joint_lower_limit}" upper="${elbow_joint_upper_limit}" />
+        <origin xyz="${fore_arm_x} ${fore_arm_y} ${fore_arm_z}" rpy="${fore_arm_roll} ${fore_arm_pitch} ${fore_arm_yaw}"/>
+    </joint>
+    <joint name="wrist_base_joint" type="revolute">
         <parent link="fore_arm_link"/>
+        <child link="wrist_link"/>
+        <axis xyz="0 1 0" />
+        <limit effort="10" velocity="1"  lower="${wrist_joint_lower_limit}" upper="${wrist_joint_upper_limit}" />
+        <origin xyz="${wrist_x} ${wrist_y} ${wrist_z}" rpy="${wrist_roll} ${wrist_pitch} ${wrist_yaw}"/>
+      </joint>
+    <joint name="gimbal_base_joint" type="fixed">
+        <parent link="wrist_link"/>
         <child link="gimbal_base_link"/>
-        <axis xyz="0 1 0" />
-        <limit effort="10" velocity="1"  lower="${-55.0*M_PI/180.0}" upper="0.0" />
-        <origin xyz="0.0 0.0 0.3" rpy="0 ${-5.0*M_PI/180.0} 0"/>
-    </joint>
-    <link name="gimbal_base_link">
-        <visual>
-            <origin xyz="0.0 0.0 0.05" rpy="0 0 0"/>
-            <geometry>
-                <cylinder length="0.10" radius="0.03"/>
-            </geometry>
-            <material name="white"/>
-        </visual>
-        <collision>
-            <origin xyz="0.0 0.0 0.0" rpy="0 0 0"/>
-            <geometry>
-                <cylinder length="0.10" radius="0.03"/>
-            </geometry>
-        </collision>
-    </link>
+        <origin xyz="0.0 0.0 0.05" rpy="0 0 0"/>
+    </joint>
     <joint name="main_cam_base_joint" type="prismatic">
         <parent link="gimbal_base_link"/>

Commit message: update: update description, control node and launch files for robot_state_publisher
Signed-off-by: Jaeyoung Lee <jylee0121@gmail.com>

File: nesfr_arm_description/urdf/nesfr_arm.urdf.xacro (robot description, xacro)
@@ -140,5 +140,5 @@
         <origin xyz="${fore_arm_x} ${fore_arm_y} ${fore_arm_z}" rpy="${fore_arm_roll} ${fore_arm_pitch} ${fore_arm_yaw}"/>
     </joint>
-    <joint name="wrist_base_joint" type="revolute">
+    <joint name="wrist_joint" type="revolute">
         <parent link="fore_arm_link"/>
         <child link="wrist_link"/>

Commit message: update: use prefix for robot_description urdf
Signed-off-by: Jaeyoung Lee <jylee0121@gmail.com>

File: nesfr_arm_description/urdf/nesfr_arm.urdf.xacro (robot description, xacro)
@@ -2,4 +2,6 @@
 <robot xmlns:xacro="http://wiki.ros.org/xacro" name="nesfr_arm" >
     <xacro:property name="M_PI" value="3.1415926535897931" />
+    <xacro:arg name="prefix" default=""/>
+    <xacro:property name="prefix" value="$(arg prefix)"/>
     <!--
       reference: https://answers.ros.org/question/401950/ros2-any-idea-on-how-to-pass-parameters-yaml-to-a-xacro-file-via-launch-python-script/
@@ -60,37 +62,37 @@
         <color rgba="0.1 0.1 0.1 1" />
     </material>
-    <link name="base_link"/>
-    <link name="robot_arm_base_link"/>
-    <link name="upper_arm_link">
-        <visual>
-            <origin xyz="0.0 0.0 0.15" rpy="0 0 0"/>
-            <geometry>
-                <box size="0.05 0.05 0.3" />
-            </geometry>
-            <material name="white"/>
-        </visual>
-        <collision>
-            <origin xyz="0.0 0.0 0.15" rpy="0 0 0"/>
-            <geometry>
-                <box size="0.05 0.05 0.3" />
-            </geometry>
-        </collision>
-    </link>
-    <link name="fore_arm_link">
-        <visual>
-            <origin xyz="0.0 0.0 0.15" rpy="0 0 0"/>
-            <geometry>
-                <box size="0.05 0.05 0.3" />
-            </geometry>
-            <material name="white"/>
-        </visual>
-        <collision>
-            <origin xyz="0.0 0.0 0.15" rpy="0 0 0"/>
-            <geometry>
-                <box size="0.05 0.05 0.3" />
-            </geometry>
-        </collision>
-    </link>
-    <link name="wrist_link">
+    <link name="${prefix}base_link"/>
+    <link name="${prefix}robot_arm_base_link"/>
+    <link name="${prefix}upper_arm_link">
+        <visual>
+            <origin xyz="0.0 0.0 0.15" rpy="0 0 0"/>
+            <geometry>
+                <box size="0.05 0.05 0.3" />
+            </geometry>
+            <material name="white"/>
+        </visual>
+        <collision>
+            <origin xyz="0.0 0.0 0.15" rpy="0 0 0"/>
+            <geometry>
+                <box size="0.05 0.05 0.3" />
+            </geometry>
+        </collision>
+    </link>
+    <link name="${prefix}fore_arm_link">
+        <visual>
+            <origin xyz="0.0 0.0 0.15" rpy="0 0 0"/>
+            <geometry>
+                <box size="0.05 0.05 0.3" />
+            </geometry>
+            <material name="white"/>
+        </visual>
+        <collision>
+            <origin xyz="0.0 0.0 0.15" rpy="0 0 0"/>
+            <geometry>
+                <box size="0.05 0.05 0.3" />
+            </geometry>
+        </collision>
+    </link>
+    <link name="${prefix}wrist_link">
         <visual>
             <origin xyz="0.0 0.0 0.025" rpy="0 0 0"/>
@@ -107,5 +109,5 @@
         </collision>
       </link>
-    <link name="gimbal_base_link">
+    <link name="${prefix}gimbal_base_link">
         <visual>
             <origin xyz="0.0 0.0 0.05" rpy="0 0 0"/>
@@ -122,37 +124,37 @@
         </collision>
     </link>
-    <joint name="base-robot_arm_base_fixed_joint" type="fixed">
-        <parent link="base_link"/>
-        <child link="robot_arm_base_link"/>
-    </joint>
-    <joint name="shoulder_lift" type="revolute">
-        <parent link="robot_arm_base_link"/>
-        <child link="upper_arm_link"/>
+    <joint name="${prefix}base-robot_arm_base_fixed_joint" type="fixed">
+        <parent link="${prefix}base_link"/>
+        <child link="${prefix}robot_arm_base_link"/>
+    </joint>
+    <joint name="${prefix}shoulder_lift" type="revolute">
+        <parent link="${prefix}robot_arm_base_link"/>
+        <child link="${prefix}upper_arm_link"/>
         <axis xyz="0 1 0" />
         <limit effort="10" velocity="1"  lower="${shoulder_lift_lower_limit}" upper="${shoulder_lift_upper_limit}" />
         <origin xyz="${upper_arm_x} ${upper_arm_y} ${upper_arm_z}" rpy="${upper_arm_roll} ${upper_arm_pitch} ${upper_arm_yaw}"/>
     </joint>
-    <joint name="elbow_joint" type="revolute">
-        <parent link="upper_arm_link"/>
-        <child link="fore_arm_link"/>
+    <joint name="${prefix}elbow_joint" type="revolute">
+        <parent link="${prefix}upper_arm_link"/>
+        <child link="${prefix}fore_arm_link"/>
         <axis xyz="0 1 0" />
         <limit effort="10" velocity="1"  lower="${elbow_joint_lower_limit}" upper="${elbow_joint_upper_limit}" />
         <origin xyz="${fore_arm_x} ${fore_arm_y} ${fore_arm_z}" rpy="${fore_arm_roll} ${fore_arm_pitch} ${fore_arm_yaw}"/>
     </joint>
-    <joint name="wrist_joint" type="revolute">
-        <parent link="fore_arm_link"/>
-        <child link="wrist_link"/>
+    <joint name="${prefix}wrist_joint" type="revolute">
+        <parent link="${prefix}fore_arm_link"/>
+        <child link="${prefix}wrist_link"/>
         <axis xyz="0 1 0" />
         <limit effort="10" velocity="1"  lower="${wrist_joint_lower_limit}" upper="${wrist_joint_upper_limit}" />
         <origin xyz="${wrist_x} ${wrist_y} ${wrist_z}" rpy="${wrist_roll} ${wrist_pitch} ${wrist_yaw}"/>
       </joint>
-    <joint name="gimbal_base_joint" type="fixed">
-        <parent link="wrist_link"/>
-        <child link="gimbal_base_link"/>
+    <joint name="${prefix}gimbal_base_joint" type="fixed">
+        <parent link="${prefix}wrist_link"/>
+        <child link="${prefix}gimbal_base_link"/>
         <origin xyz="0.0 0.0 0.05" rpy="0 0 0"/>
     </joint>
-    <joint name="main_cam_base_joint" type="prismatic">
-        <parent link="gimbal_base_link"/>
-        <child link="main_cam_pan_link"/>
+    <joint name="${prefix}main_cam_base_joint" type="prismatic">
+        <parent link="${prefix}gimbal_base_link"/>
+        <child link="${prefix}main_cam_pan_link"/>
         <axis xyz="0 0 1" />
         <limit effort="10" velocity="1"  lower="0.0" upper="2.0" />
@@ -162,23 +164,23 @@
         Main Camera
     -->
-    <link name="main_cam_pan_link">
-    </link>
-    <joint name="main_cam_pan_joint" type="revolute">
-        <parent link="main_cam_pan_link"/>
-        <child link="main_cam_tilt_link"/>
+    <link name="${prefix}main_cam_pan_link">
+    </link>
+    <joint name="${prefix}main_cam_pan_joint" type="revolute">
+        <parent link="${prefix}main_cam_pan_link"/>
+        <child link="${prefix}main_cam_tilt_link"/>
         <axis xyz="0 0 1" />
         <limit effort="10" velocity="1"  lower="-${M_PI}" upper="${M_PI}" />
         <origin xyz="0.0 0.0 0.0" rpy="0 0 0"/>
     </joint>
-    <link name="main_cam_tilt_link">
-    </link>
-    <joint name="main_cam_tilt_joint" type="revolute">
-        <parent link="main_cam_tilt_link"/>
-        <child link="main_cam_link"/>
+    <link name="${prefix}main_cam_tilt_link">
+    </link>
+    <joint name="${prefix}main_cam_tilt_joint" type="revolute">
+        <parent link="${prefix}main_cam_tilt_link"/>
+        <child link="${prefix}main_cam_link"/>
         <axis xyz="0 1 0" />
         <limit effort="10" velocity="1"  lower="-${0.5*M_PI}" upper="${0.5*M_PI}" />
         <origin xyz="0.0 0.0 0.0" rpy="0 0 0"/>
     </joint>
-    <link name="main_cam_link">
+    <link name="${prefix}main_cam_link">
         <visual>
             <origin xyz="0.0 0.0 ${0.5*main_cam_size_z}" rpy="0 0 0"/>
@@ -195,10 +197,10 @@
         </collision>
     </link>
-    <joint name="main_img_joint" type="fixed">
-        <parent link="main_cam_link"/>
-        <child link="main_img_link"/>
+    <joint name="${prefix}main_img_joint" type="fixed">
+        <parent link="${prefix}main_cam_link"/>
+        <child link="${prefix}main_img_link"/>
         <origin xyz="0.0 0.0 0.0" rpy="-${0.5*M_PI} 0 -${0.5*M_PI}"/>
     </joint>
-    <link name="main_img_link">
+    <link name="${prefix}main_img_link">
     </link>
 </robot>
