Commit message: update: split into nesfr7_arm and nesfr7_arm_only
Signed-off-by: Jaeyoung Lee <jylee0121@gmail.com>

File: nesfr_arm_description/urdf/nesfr_arm.urdf.xacro (robot description, xacro)
@@ -16,4 +16,10 @@
     <xacro:property name="wrist_joint_lower_limit" value="${nesfr_arm_parameters['joint_limits']['wrist_joint']['min_position']}"/>
     <xacro:property name="wrist_joint_upper_limit" value="${nesfr_arm_parameters['joint_limits']['wrist_joint']['max_position']}"/>
+    <xacro:property name="robot_arm_base_x" value="${nesfr_arm_parameters['kinematics']['robot_arm_base']['x']}" />
+    <xacro:property name="robot_arm_base_y" value="${nesfr_arm_parameters['kinematics']['robot_arm_base']['y']}" />
+    <xacro:property name="robot_arm_base_z" value="${nesfr_arm_parameters['kinematics']['robot_arm_base']['z']}" />
+    <xacro:property name="robot_arm_base_roll" value="${nesfr_arm_parameters['kinematics']['robot_arm_base']['roll']}" />
+    <xacro:property name="robot_arm_base_pitch" value="${nesfr_arm_parameters['kinematics']['robot_arm_base']['pitch']}" />
+    <xacro:property name="robot_arm_base_yaw" value="${nesfr_arm_parameters['kinematics']['robot_arm_base']['yaw']}" />
     <xacro:property name="upper_arm_x" value="${nesfr_arm_parameters['kinematics']['upper_arm']['x']}" />
     <xacro:property name="upper_arm_y" value="${nesfr_arm_parameters['kinematics']['upper_arm']['y']}" />
@@ -28,10 +34,4 @@
     <xacro:property name="fore_arm_pitch" value="${nesfr_arm_parameters['kinematics']['fore_arm']['pitch']}" />
     <xacro:property name="fore_arm_yaw" value="${nesfr_arm_parameters['kinematics']['fore_arm']['yaw']}" />
-    <xacro:property name="upper_arm_x" value="${nesfr_arm_parameters['kinematics']['upper_arm']['x']}" />
-    <xacro:property name="upper_arm_y" value="${nesfr_arm_parameters['kinematics']['upper_arm']['y']}" />
-    <xacro:property name="upper_arm_z" value="${nesfr_arm_parameters['kinematics']['upper_arm']['z']}" />
-    <xacro:property name="upper_arm_roll" value="${nesfr_arm_parameters['kinematics']['upper_arm']['roll']}" />
-    <xacro:property name="upper_arm_pitch" value="${nesfr_arm_parameters['kinematics']['upper_arm']['pitch']}" />
-    <xacro:property name="upper_arm_yaw" value="${nesfr_arm_parameters['kinematics']['upper_arm']['yaw']}" />
     <xacro:property name="wrist_x" value="${nesfr_arm_parameters['kinematics']['wrist']['x']}" />
     <xacro:property name="wrist_y" value="${nesfr_arm_parameters['kinematics']['wrist']['y']}" />
@@ -127,4 +127,5 @@
         <parent link="${prefix}base_link"/>
         <child link="${prefix}robot_arm_base_link"/>
+        <origin xyz="${robot_arm_base_x} ${robot_arm_base_y} ${robot_arm_base_z}" rpy="${robot_arm_base_roll} ${robot_arm_base_pitch} ${robot_arm_base_yaw}"/>
     </joint>
     <joint name="${prefix}shoulder_lift" type="revolute">

Commit message: fix: fix urdf.xacro for humble
Signed-off-by: Jaeyoung Lee <jylee0121@gmail.com>

File: nesfr_arm_description/urdf/nesfr_arm.urdf.xacro (robot description, xacro)
@@ -9,5 +9,5 @@
     <xacro:arg name="nesfr_arm_params" default=""/>
     <xacro:property name="nesfr_arm_params_file" value="$(arg nesfr_arm_params)"/>
-    <xacro:property name="nesfr_arm_parameters" value="${load_yaml(nesfr_arm_params_file)}"/>
+    <xacro:property name="nesfr_arm_parameters" value="${xacro.load_yaml(nesfr_arm_params_file)}"/>
     <xacro:property name="shoulder_lift_lower_limit" value="${nesfr_arm_parameters['joint_limits']['shoulder_lift']['min_position']}"/>
     <xacro:property name="shoulder_lift_upper_limit" value="${nesfr_arm_parameters['joint_limits']['shoulder_lift']['max_position']}"/>
